File: acadapter.kicad_sch (KiCad schematic)
At the start: 11 parts, among them J1 Conn_01x04, J2 USB_C_Receptacle_USB2.0, Q1 2N3904, Q2 2N3904, U1 AP7380-50W5-7

Commit message: add license to readme. update part numbers
Parts:
- C1, C2: DK (none) -> 490-10014-1-ND; PARTNO (none) -> GRM155C81E105KE11D
- J2: DK (none) -> 2073-USB4105-GF-ACT-ND
- Q2: DK (none) -> MMBT3904TPMSCT-ND; PARTNO (none) -> MMBT3904-TP
- R1, R2, R3: DK (none) -> 311-10KJRCT-ND; PARTNO (none) -> RC0402JR-0710KL
- R4: DK (none) -> 311-4.7KLRCT-ND; PARTNO (none) -> RC0402FR-074K7L
Changed lines of the file:
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@@
+			)
+		)
+		(property "DK" "311-10KJRCT-ND"
+			(at 68.58 72.39 0)
+			(effects
+				(font
+					(size 1.27 1.27)
+				)
+				(hide yes)
+			)
+		)
+		(property "PARTNO" "RC0402JR-0710KL"
+			(at 68.58 72.39 0)
+			(effects
+				(font
+					(size 1.27 1.27)
+				)
+				(hide yes)
 			)
 		)
@@
 			)
 		)
+		(property "DK" "311-10KJRCT-ND"
+			(at 74.93 87.63 90)
+			(effects
+				(font
+					(size 1.27 1.27)
+				)
+				(hide yes)
+			)
+		)
+		(property "PARTNO" "RC0402JR-0710KL"
+			(at 74.93 87.63 90)
+			(effects
+				(font
+					(size 1.27 1.27)
+				)
+				(hide yes)
+			)
+		)
 		(pin "2"
 		)
@@
 			)
 		)
+		(property "DK" "311-10KJRCT-ND"
+			(at 88.9 72.39 0)
+			(effects
+				(font
+					(size 1.27 1.27)
+				)
+				(hide yes)
+			)
+		)
+		(property "PARTNO" "RC0402JR-0710KL"
+			(at 88.9 72.39 0)
+			(effects
+				(font
+					(size 1.27 1.27)
+				)
+				(hide yes)
+			)
+		)
 		(pin "2"
 		)
@@
 			)
 		)
+		(property "DK" "311-4.7KLRCT-ND"
+			(at 101.6 78.74 90)
+			(effects
+				(font
+					(size 1.27 1.27)
+				)
+				(hide yes)
+			)
+		)
+		(property "PARTNO" "RC0402FR-074K7L"
+			(at 101.6 78.74 90)
+			(effects
+				(font
+					(size 1.27 1.27)
+				)
+				(hide yes)
+			)
+		)
 		(pin "2"
 		)
@@
 			)
 		)
+		(property "DK" "490-10014-1-ND"
+			(at 77.47 45.72 0)
+			(effects
+				(font
+					(size 1.27 1.27)
+				)
+				(hide yes)
+			)
+		)
+		(property "PARTNO" "GRM155C81E105KE11D"
+			(at 77.47 45.72 0)
+			(effects
+				(font
+					(size 1.27 1.27)
+				)
+				(hide yes)
+			)
+		)
 		(pin "2"
 		)
@@
 			)
 		)
+		(property "DK" "MMBT3904TPMSCT-ND"
+			(at 111.76 78.74 0)
+			(effects
+				(font
+					(size 1.27 1.27)
+				)
+				(hide yes)
+			)
+		)
+		(property "PARTNO" "MMBT3904-TP"
+			(at 111.76 78.74 0)
+			(effects
+				(font
+					(size 1.27 1.27)
+				)
+				(hide yes)
+			)
+		)
 		(pin "2"
 		)
@@
 			)
 		)
+		(property "DK" "490-10014-1-ND"
+			(at 104.14 45.72 0)
+			(effects
+				(font
+					(size 1.27 1.27)
+				)
+				(hide yes)
+			)
+		)
+		(property "PARTNO" "GRM155C81E105KE11D"
+			(at 104.14 45.72 0)
+			(effects
+				(font
+					(size 1.27 1.27)
+				)
+				(hide yes)
+			)
+		)
 		(pin "2"
 		)
@@
 			)
 		)
-		(property "DK" ""
+		(property "DK" "2073-USB4105-GF-ACT-ND"
 			(at 151.13 68.58 0)
 			(effects
